File: CODEC.sch (KiCad schematic (older format))
At the start: 47 parts, among them J701 AUEXT, J702 RIN, J703 LIN/MONO, J704 ROUT, J705 LOUT, U701 WM8731, U702 TL074, Y701 11.289600MHz

Commit message: current
Connections:
- net GND: now also J702.2
- net at J703.1, R706.2: no longer J702.2
Changed lines of the file:
@@
 Title "ESP32 Eurorack Audio Module"
 Date "2019-03-27"
-Rev "B2-public"
+Rev "C"
 Comp "(c) Robert Manzke 2019"
 Comment1 "https://creativecommons.org/licenses/by-nc-sa/4.0/"
@@
 Wire Wire Line
 	7350 1400 7100 1400
-Wire Wire Line
-	7350 2850 7250 2850
-Wire Wire Line
-	7250 2850 7250 1500
-Wire Wire Line
-	7250 1500 7100 1500
 $Comp
 L jack_2p:JACK_2P J?
@@
 	1    0    0    1
 $EndComp
-Wire Wire Line
-	7250 2850 7100 2850
-Connection ~ 7250 2850
 $Comp
 L power:GND #PWR0706
@@
 Wire Notes Line
 	2350 550  500  550
+Wire Wire Line
+	7100 2850 7350 2850
+Wire Wire Line
+	7100 1500 7150 1500
+Wire Wire Line
+	7150 1500 7150 1650
+Connection ~ 7150 1650
 $EndSCHEMATC
